File: Hardware/stm32g030c8t6/stm32g030c8t6.brd (EAGLE design)
At the start: 63 x 22.9 mm, 27 parts, among them IC1 STM32G030C8T6, IC2 AP2114HA-3.3TRG1, J1 USB_MINI-B_SMT, Y1 DSC6083CI1A-350K000T

Commit message: Added pullup to RX pin
Parts:
- added JP6: JUMPER-SMT_2_NC_PASTE_SILK, SparkFun-Jumpers:SMT-JUMPER_2_NC_PASTE_SILK
- added R5: 1.8K, rcl:R0805
Connections:
- new net N$1: JP6.2, R5.1
- net +3V3: now also R5.2
- net PA10-U1RX: now also J3.19, JP6.1; no longer J3.17
- net PC6: now also J3.18; no longer J3.19
- net PC7: now also J3.17; no longer J3.18
Routing:
- net +3V3: track 142.3 -> 151.2 mm, vias 6 -> 7
- net PA10-U1RX: track 35.4 -> 40.9 mm
- net N$1: track 0.00 -> 2.45 mm
- net PC7: track 6.54 -> 7.28 mm
- net GND: track 138.6 -> 139.3 mm
